File: 36V 3.6A 30D/CAN-Controlled/Hardware/PowerServo AE 36V 3.6A 30D.kicad_pcb (KiCad board)
At the start: 4 copper layers, 35.7 x 35.5 mm, 36 parts, among them IC1 DRV8251DDAR, J1 Control_In, J2 MOT_A, J3 Prog_IN, J4 Power_In, J5 Power_In, J6 Control_In, J7 MOT_B, U1 LMZM23601V5, U2 TLV76733DRVx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

Commit message: various
Parts:
- C1, C11: value 100nF -> 100nF, X7R
- C2: value 10uF -> 10uF, 50V, X7R
- C5: value 1uF -> 1uF, X7R
- C6: value 2.2uF -> 2.2uF, X7R
- C7: value 10uF -> 10uF, 50V
- C8: value 100nF -> 100nF, 50V
- moved C2 6.95 mm to (108.0, 77.5), turned to 180 degrees
Connections:
- U1 pad 4: GND -> +12V
Routing:
- net GND: track 27.3 -> 23.7 mm, vias 152 -> 150
- net +12V: track 6.89 -> 4.70 mm
Changed lines of the file:
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@@
 			)
 		)
-		(property "Value" "10uF"
+		(property "Value" "10uF, 50V"
 			(at -0.000001 -1.85 -90)
 			(layer "B.Fab")
@@
 	(footprint "Capacitor_SMD:C_1206_3216Metric"
 		(layer "B.Cu")
-		(at 106.25 70.775 -90)
+		(at 108 77.5 180)
 		(descr "Capacitor SMD 1206 (3216 Metric), square (rectangular) end terminal, IPC_7351 nominal, (Body size source: IPC-SM-782 page 76, https://www.pcb-3d.com/wordpress/wp-content/uploads/ipc-sm-782a_amendment_1_and_2.pdf), generated with kicad-footprint-generator")
 		(tags "capacitor")
 		(property "Reference" "C2"
-			(at 2.475 1.75 90)
+			(at 2.475 1.75 360)
 			(layer "B.SilkS")
 			(effects
@@
 			)
 		)
-		(property "Value" "10uF"
-			(at -0.000001 -1.85 90)
+		(property "Value" "10uF, 50V, X7R"
+			(at -0.000001 -1.85 360)
 			(layer "B.Fab")
 			(effects
@@
 		)
 		(property "Footprint" "Capacitor_SMD:C_1206_3216Metric"
-			(at 0 0 90)
+			(at 0 0 0)
 			(unlocked yes)
 			(layer "B.Fab")
@@
 		)
 		(property "Datasheet" ""
-			(at 0 0 90)
+			(at 0 0 0)
 			(unlocked yes)
 			(layer "B.Fab")
@@
 		)
 		(property "Description" "Unpolarized capacitor"
-			(at 0 0 90)
+			(at 0 0 0)
 			(unlocked yes)
 			(layer "B.Fab")
@@
 		)
 		(fp_line
-			(start -2.3 1.150001)
-			(end -2.3 -1.150001)
+			(start 2.3 1.150001)
+			(end -2.3 1.150001)
 			(stroke
 				(width 0.05)
@@
 		)
 		(fp_line
-			(start 2.3 1.150001)
-			(end -2.3 1.150001)
+			(start 2.3 -1.150001)
+			(end 2.3 1.150001)
 			(stroke
 				(width 0.05)
@@
 		)
 		(fp_line
-			(start -2.3 -1.150001)
-			(end 2.3 -1.150001)
+			(start -2.3 1.150001)
+			(end -2.3 -1.150001)
 			(stroke
 				(width 0.05)
@@
 		)
 		(fp_line
-			(start 2.3 -1.150001)
-			(end 2.3 1.150001)
+			(start -2.3 -1.150001)
+			(end 2.3 -1.150001)
 			(stroke
 				(width 0.05)
@@
 		)
 		(fp_line
-			(start 1.600001 0.800001)
+			(start 1.6 0.800004)
 			(end -1.6 0.8)
 			(stroke
@@
 		)
 		(fp_line
-			(start -1.6 0.8)
-			(end -1.600001 -0.800001)
+			(start 1.6 -0.8)
+			(end 1.6 0.800004)
 			(stroke
 				(width 0.1)
@@
 		)
 		(fp_line
-			(start 1.6 -0.8)
-			(end 1.600001 0.800001)
+			(start -1.6 0.8)
+			(end -1.6 -0.800004)
 			(stroke
 				(width 0.1)
@@
 		)
 		(fp_line
-			(start -1.600001 -0.800001)
+			(start -1.6 -0.800004)
 			(end 1.6 -0.8)
 			(stroke
@@
 		)
 		(fp_text user "${REFERENCE}"
-			(at 0 0 90)
+			(at 0 0 360)
 			(layer "B.Fab")
 			(effects
@@
 		)
 		(pad "1" smd roundrect
-			(at -1.475 0 270)
+			(at -1.475 0 180)
 			(size 1.15 1.8)
 			(layers "B.Cu" "B.Paste" "B.Mask")
@@
 		)
 		(pad "2" smd roundrect
-			(at 1.475 0 270)
+			(at 1.475 0 180)
 			(size 1.15 1.8)
 			(layers "B.Cu" "B.Paste" "B.Mask")
@@
 			)
 		)
-		(property "Value" "2.2uF"
+		(property "Value" "2.2uF, X7R"
 			(at 0.000002 -1.159999 -90)
 			(layer "B.Fab")
@@
 			)
 		)
-		(property "Value" "100nF"
+		(property "Value" "100nF, X7R"
 			(at -0.000001 -1.429999 90)
 			(layer "B.Fab")
@@
 			)
 		)
-		(property "Value" "100nF"
+		(property "Value" "100nF, X7R"
 			(at 0 -1.16 90)
 			(layer "B.Fab")
@@
 			)
 		)
-		(property "Value" "100nF"
+		(property "Value" "100nF, 50V"
 			(at 0.000001 -1.430001 90)
 			(layer "B.Fab")
@@
 			(layers "B.Cu" "B.Paste" "B.Mask")
 			(roundrect_rratio 0.25)
-			(net 1 "GND")
+			(net 3 "+12V")
 			(pinfunction "EN")
 			(pintype "input")
@@
 			)
 		)
-		(property "Value" "1uF"
+		(property "Value" "1uF, X7R"
 			(at 0.000002 -1.159999 90)
 			(layer "B.Fab")
@@
 	)
 	(via
-		(at 108 77)
-		(size 0.9)
-		(drill 0.6)
-		(layers "F.Cu" "B.Cu")
-		(free yes)
-		(net 1)
-	)
-	(via
 		(at 92.5 82.75)
 		(size 0.6)
@@
 	)
 	(via
-		(at 108 78)
-		(size 0.9)
-		(drill 0.6)
-		(layers "F.Cu" "B.Cu")
-		(free yes)
-		(net 1)
-	)
-	(via
 		(at 94 73.25)
 		(size 0.6)
@@
 	)
 	(segment
-		(start 106.25 69.3)
-		(end 106.25 67.15)
-		(width 0.508)
-		(layer "B.Cu")
-		(net 1)
-	)
-	(segment
 		(start 100.25 80.02)
 		(end 100.127 79.897)
@@
 	)
 	(segment
-		(start 103.425001 81.28)
-		(end 103.854999 80.850002)
-		(width 0.5)
-		(layer "B.Cu")
-		(net 1)
-	)
-	(segment
 		(start 104.525001 79.65)
 		(end 103.605002 79.65)
@@
 	)
 	(segment
-		(start 103.854999 80.850002)
-		(end 104.775 80.850002)
-		(width 0.4)
-		(layer "B.Cu")
-		(net 1)
-	)
-	(segment
 		(start 106.25 67.15)
 		(end 106.4 67)
@@
 	)
 	(segment
-		(start 103.848427 71.562486)
-		(end 105.312486 71.562486)
-		(width 0.762)
+		(start 104.525 80.25)
+		(end 104.525 80.850002)
+		(width 0.5)
 		(layer "B.Cu")
 		(net 3)
@@
 		(width 0.762)
 		(layer "B.Cu")
-		(net 3)
-	)
-	(segment
-		(start 105.312486 71.562486)
-		(end 106.25 72.5)
-		(width 0.762)
-		(layer "B.Cu")
