File: 1. Little Boy (4.1A @ 36V)/1. Hardware/_autosave-PowerServo AE 36V 3.6A 30D.kicad_sch (KiCad schematic)
At the start: 32 parts, among them IC1 DRV8251DDAR, J1 Control_In, J2 MOT_A, J3 Prog_IN, J4 Power_In, J5 Power_In, J6 Control_In, J7 MOT_B, U1 LMZM23601V5, U2 TLV76733DRVx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

Commit message: 3
Parts:
- R1: value 300 -> 15k
Changed lines of the file:
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@@
 			)
 		)
-		(property "Value" "300"
+		(property "Value" "15k"
 			(at 154.686 149.86 90)
 			(effects
