File: 2. Little Boy - External (4.1A @ 36V)/1. Hardware/Little Boy - External.kicad_sch (KiCad schematic)
At the start: 76 parts, among them IC1 DRV8251DDAR, IC2 AS5600-ASOT, J1 Conn_01x01, J10 MOT_B, J11 MOT_A, J12 Conn_01x01, J13 Control_In, J14 Control_In, J15 Conn_01x06_MountingPin, J16 Conn_01x06_MountingPin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

Commit message: 3
Parts:
- J1: footprint TestPoint:TestPoint_THTPad_1.0x1.0mm_Drill0.5mm -> Connector_PinHeader_2.54mm:PinHeader_1x01_P2.54mm_Vertical
Other:
- moved on the sheet: C1, C10, C2, C3, C4, C5, C6, C7, C8, C9, D1, D2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
