File: 2. Little Boy - External (4.1A @ 36V)/1. Hardware/Little Boy - External.kicad_sch (KiCad schematic)
At the start: 83 parts, among them J1 TESTPOINT, J10 MOT_B, J11 MOT_A, J12 TESTPOINT, J13 Control_In, J14 Control_In, J15 Conn_01x06_MountingPin, J16 Conn_01x06_MountingPin, J17 TESTPOINT, J2 TESTPOINT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

Commit message: v4 full
Other:
- moved on the sheet: C10, C11, C12, C13, C23, C8, J10, J11, J15, J17, J4, J6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
