File: 2. Little Boy - External (4.1A @ 36V)/1. Hardware/Little Boy - External.kicad_sch (KiCad schematic)
At the start: 50 parts, among them IC1 DRV8251DDAR, IC2 AS5600-ASOT, J1 Prog_IN, J10 I2C IN, J2 SPI_OUT, J3 Power_In, J4 Power_In, J5 MOT_B, J6 MOT_A, J7 SPI_IN, J8 Control_In, J9 Control_In, U1 STM32G0B1CBTx, U2 LMR33630CDDA, U3 TLV76733DRVx, U4 TJA1051T-3, U5 MA730, Y1 Crystal_GND24

Commit message: V2 init commit
Parts:
- removed J10: I2C IN, symbol Connector_Generic:Conn_01x06
- removed J2: SPI_OUT, symbol Connector_Generic:Conn_01x06
- removed J7: SPI_IN, symbol Connector_Generic:Conn_01x06
- added H1, H10, H11, H12, H2, H3, H4, H5, H6, H7, H8, H9: MountingHole, MountingHole:MountingHole_2.2mm_M2, symbol Mechanical:MountingHole
- added J10, J11, J7: Conn_01x06_MountingPin, Connector_FFC-FPC:Hirose_FH12-6S-0.5SH_1x06-1MP_P0.50mm_Horizontal, symbol Connector_Generic_MountingPin:Conn_01x06_MountingPin
- added R8: 900, Resistor_SMD:R_0402_1005Metric, symbol Device:R
- C10, C13, C18, C9: footprint Capacitor_SMD:C_0402_1005Metric -> Capacitor_SMD:C_0805_2012Metric
- C11: footprint Capacitor_SMD:C_1206_3216Metric -> Capacitor_SMD:C_0805_2012Metric
- C12, C14: footprint Capacitor_SMD:C_0603_1608Metric -> Capacitor_SMD:C_0402_1005Metric
- C16, C17: footprint Capacitor_SMD:C_0402_1005Metric -> Capacitor_SMD:C_0603_1608Metric
- D1, D2: footprint LED_SMD:LED_0402_1005Metric -> LED_SMD:LED_0603_1608Metric
- IC1: footprint _custom:SOIC127P600X170-9N -> KiCadLibrary:SOIC127P600X170-9N
- IC2: footprint custom:SOIC127P600X175-8N -> KiCadLibrary:SOIC127P600X175-8N
- L2: footprint (none) -> Inductor_SMD:L_1008_2520Metric
- R6: value 24.9k -> 24k; footprint Resistor_SMD:R_0402_1005Metric -> Resistor_SMD:R_0603_1608Metric
- Y1: footprint (none) -> Crystal:Crystal_SMD_3225-4Pin_3.2x2.5mm
Connections:
- net +3.3V: now also J11.6 (Pin_6); no longer L1.1
- net +3.3VP: now also J7.6 (Pin_6)
- net +3V3: now also L1.1, J10.6 (Pin_6)
- net DRV_IN1: now also U1.28 (PA8); no longer U1.29 (PA9/UCPD1_DBCC1)
- net DRV_IN2: now also U1.29 (PA9/UCPD1_DBCC1); no longer U1.28 (PA8)
- net Encoder_SCL: now also J7.2 (Pin_2)
- net Encoder_SDA: now also J7.4 (Pin_4)
- net GND: now also J10.3 (Pin_3), J10.MP (MountPin), R8.1; no longer C20.1, R6.1
- net GND1: now also C20.1, J11.3 (Pin_3), J11.MP (MountPin)
- net GND2: now also J7.3 (Pin_3), J7.MP (MountPin)
- net MAG_CS: now also J10.1 (Pin_1)
- net MISO: now also J10.4 (Pin_4)
- net MOSI: now also J10.5 (Pin_5)
- net RP_RX: now also U1.47 (PB8); no longer U1.19 (PB0)
- net RP_TX: now also U1.48 (PB9); no longer U1.20 (PB1)
- net SCK: now also J10.2 (Pin_2)
- net  MOT_A: now reaches IC1.6 (OUT1), J6.1 (Pin_1)
- net at R2.1: now also U1.13 (PA2); no longer U1.47 (PB8)
- net at R3.1: now also U1.14 (PA3); no longer U1.48 (PB9)
- net at U5.4 (MOSI): now also J11.1 (Pin_1)
- net at U5.7 (MISO): now also J11.2 (Pin_2)
- net at U5.12 (SCLK): now also J11.4 (Pin_4)
- net at U5.5 (~{CS}): now also J11.5 (Pin_5)
- new net: R6.1, R8.2
Other:
- note added: "ENCODER 2"
- note added: "POWER"
- moved on the sheet: C1, C10, C13, C15, C16, C17, C18, C19, C2, C20, C3, C4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

Commit message: Esthetic Changes, Fix-up of daughter boards.
Parts:
- added C21: 100nF, Capacitor_SMD:C_1206_3216Metric, symbol Device:C
- added C22, C23, C24: 100nF, Capacitor_SMD:C_0402_1005Metric, symbol Device:C
- added R10, R9: 4.7k, Resistor_SMD:R_0402_1005Metric, symbol Device:R
Connections:
- net +3.3VP: now also C23.1, R10.2, R9.2
- net +3V3: now also C21.1, C22.1, C24.1
- net Encoder_SCL: now also R9.1
- net Encoder_SDA: now also R10.1
- net GND: now also C21.2, C22.2, C24.2
- net GND2: now also C23.2
- net at J11.1 (Pin_1): now also U5.5 (~{CS}); no longer U5.4 (MOSI)
- net at J11.2 (Pin_2): now also U5.12 (SCLK); no longer U5.7 (MISO)
- net at J11.4 (Pin_4): now also U5.7 (MISO); no longer U5.12 (SCLK)
- net at J11.5 (Pin_5): now also U5.4 (MOSI); no longer U5.5 (~{CS})

Commit message: V2.2 - Added Test Points, fixed DFM Errors
Parts:
- added J1, J12, J17, J2, J3, J6, J7: Conn_01x01, TestPoint:TestPoint_THTPad_1.0x1.0mm_Drill0.5mm, symbol Connector_Generic:Conn_01x01
- renumbered C8 to C10, C14 to C13, C9 to C14, C10 to C15, C13 to C16, C24 to C17, C15 to C18, C16 to C19, C17 to C20, C18 to C21, C19 to C22, C20 to C24, C21 to C8, C22 to C9, D2 to D1, D1 to D2, H8 to H1, H3 to H10, H12 to H11, H4 to H12, H1 to H2, H7 to H3, H9 to H4, H2 to H5, H10 to H6, H6 to H7, H5 to H8, H11 to H9, J5 to J10, J6 to J11, J8 to J13, J9 to J14, J7 to J15, J11 to J16, J1 to J4, J10 to J5, J3 to J8, J4 to J9, R8 to R7, R7 to R8, U4 to U3, U3 to U4
Connections:
- net +3V3: now also J1.1 (Pin_1), J2.1 (Pin_1), J3.1 (Pin_1)
- net +5V: now also J12.1 (Pin_1)
- net DRV_IN1: now also J7.1 (Pin_1)
- net DRV_IN2: now also J6.1 (Pin_1)
- net ISEN: now also J17.1 (Pin_1)

Commit message: review request, v0.3
Parts:
- removed C8: 100nF, Capacitor_SMD:C_1206_3216Metric, symbol Device:C
- added C25: 100nF, Capacitor_SMD:C_0402_1005Metric, symbol Device:C
- added R11: 10k, Resistor_SMD:R_0402_1005Metric, symbol Device:R
- added R12: 100k, Resistor_SMD:R_0402_1005Metric, symbol Device:R
- added U6: W25Q128JVS, Package_SO:SOIC-8_5.23x5.23mm_P1.27mm, symbol Memory_Flash:W25Q128JVS
- C11: value 10uF, 50V -> 47uF, 50V
- C18: value 100nF, 6V -> 100nF, 16V
- R4: value 15k -> 100 mOhm; footprint Resistor_SMD:R_0402_1005Metric -> Resistor_SMD:R_1206_3216Metric
Connections:
- net +12V: now also R12.2; no longer U2.3 (EN)
- net +3V3: now also C25.1, R11.1, U6.3 (IO2), U6.7 (IO3), U6.8 (VCC)
- net GND: now also C25.2, U6.4 (GND)
- net GND1: now also U5.10 (TEST)
- net FLASH_CLK: now reaches U1.25 (PB13)
- net FLASH_CLK: now also U6.6 (CLK)
- net FLASH_MISO: now reaches U1.26 (PB14)
- net FLASH_MISO: now also U6.2 (DO(IO1))
- net FLASH_MOSI: now reaches U1.32 (PA10/UCPD1_DBCC2)
- net FLASH_MOSI: now also U6.5 (DI(IO0))
- net FLASH_CS: now reaches U1.34 (PA12/PA10)
- net FLASH_CS: now also R11.2, U6.1 (~{CS})
- new net: R12.1, U2.3 (EN)
- no-connect marks 41 -> 36
Other:
- note added: "FLASH"
- moved on the sheet: C1, C10, C11, C12, C13, C14, C15, C16, C17, C18, C19, C2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

Commit message: v0.3.5 effectively, most TODOs implemented
Parts:
- removed R4: 100 mOhm, Resistor_SMD:R_1206_3216Metric, symbol Device:R
- added C8: 100uF, 80V, Capacitor_THT:CP_Radial_D8.0mm_P3.50mm, symbol Device:C_Polarized
- added R4: ERJ-B1CFR10U, Library:ERJB1_(1020), symbol _custom:ERJ-B1CFR10U
- C11: value 47uF, 50V -> 10uF, 50V
- C16: value 1uF, 6V, X7R -> 1uF, 16V, X7R
- C19, C20: value 22uF, 6V -> 22uF, 16V
- J1, J12, J17, J2, J3, J6, J7: value Conn_01x01 -> TESTPOINT; footprint TestPoint:TestPoint_THTPad_1.0x1.0mm_Drill0.5mm -> TestPoint:TestPoint_Pad_1.5x1.5mm
- JP1: value Jumper_2_Open -> Termination Jumper
- Y1: value Crystal_GND24 -> 25 MHz
- renumbered IC1 to U7, IC2 to U8
Connections:
- net +12V: now also C8.1
- net GND: now also C8.2, R4.2
- net ISEN: now also R4.1
- net  MOT_A: no longer names the net of J11.1 (Pin_1), U7.6 (OUT1)
Other:
- moved on the sheet: C24, J1, J2, R10, R11, R9

Commit message: V0.4
Parts:
- added C26, C27: 100pF, Capacitor_SMD:C_0402_1005Metric, symbol Device:C
- added FL1: ACT1210D-101-2P-TL00, _custom:ACT1210D1012PTL00, symbol Device:Filter_EMI_LL_1423
Connections:
- net CAN_H: now also C27.1, FL1.3; no longer J13.1 (Pin_1), J14.1 (Pin_1)
- net CAN_L: now also C26.2, FL1.4; no longer J13.2 (Pin_2), J14.2 (Pin_2)
- net GND: now also C26.1, C27.2
- net RP_RX: now also U3.4 (RXD); no longer U3.1 (TXD)
- net RP_TX: now also U3.1 (TXD); no longer U3.4 (RXD)
- new net: FL1.2, J13.1 (Pin_1), J14.1 (Pin_1)
- new net: FL1.1, J13.2 (Pin_2), J14.2 (Pin_2)
Other:
- moved on the sheet: C17, C25, J13, J14, JP1, R11, R8, U3, U6

Commit message: push for init manufacturing
Parts:
- C19, C20: footprint Capacitor_SMD:C_0603_1608Metric -> Capacitor_SMD:C_0805_2012Metric
- C22: value 2.2uF, X7R -> 2.2uF; footprint Capacitor_SMD:C_0402_1005Metric -> Capacitor_SMD:C_0603_1608Metric
- R2, R3: value 430 -> 470
Connections:
- net CAN_H: now also FL1.2; no longer FL1.3
- net CAN_L: now also FL1.1; no longer FL1.4
- net at J13.1 (Pin_1), J14.1 (Pin_1): now also FL1.3; no longer FL1.2
- net at J13.2 (Pin_2), J14.2 (Pin_2): now also FL1.4; no longer FL1.1
Other:
- note added: "V05: C19, C20 Bump to 0805 R2, R3 now 470 Ohm C22 Bump to 0603"
- moved on the sheet: FL1
Changed lines of the file:
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@@
 	(paper "A3")
 	(junction
+		(at 219.71 238.76)
+		(diameter 0)
+		(color 0 0 0 0)
+	)
+	(junction
 		(at 194.31 228.6)
 		(diameter 0)
@@
 	)
 	(junction
-		(at 219.71 237.49)
-		(diameter 0)
-		(color 0 0 0 0)
-	)
-	(junction
 		(at 39.37 220.98)
 		(diameter 0)
@@
 	)
 	(junction
-		(at 171.45 170.18)
+		(at 219.71 233.68)
 		(diameter 0)
 		(color 0 0 0 0)
 	)
 	(junction
-		(at 229.87 170.18)
+		(at 171.45 170.18)
 		(diameter 0)
 		(color 0 0 0 0)
 	)
 	(junction
-		(at 219.71 234.95)
+		(at 229.87 170.18)
 		(diameter 0)
 		(color 0 0 0 0)
@@
 	(wire
 		(pts
-			(xy 217.17 237.49) (xy 219.71 237.49)
-		)
-		(stroke
-			(width 0)
-			(type default)
-		)
-	)
-	(wire
-		(pts
 			(xy 264.16 104.14) (xy 257.81 104.14)
 		)
@@
 	(wire
 		(pts
-			(xy 219.71 237.49) (xy 219.71 240.03)
+			(xy 219.71 237.49) (xy 219.71 238.76)
 		)
 		(stroke
@@
 	(wire
 		(pts
-			(xy 217.17 233.68) (xy 217.17 237.49)
+			(xy 269.24 172.72) (xy 267.97 172.72)
 		)
 		(stroke
@@
 	(wire
 		(pts
-			(xy 269.24 172.72) (xy 267.97 172.72)
+			(xy 194.31 243.84) (xy 205.74 243.84)
 		)
 		(stroke
@@
 	(wire
 		(pts
-			(xy 194.31 243.84) (xy 204.47 243.84)
+			(xy 83.82 252.73) (xy 83.82 248.92)
 		)
 		(stroke
@@
 	(wire
 		(pts
-			(xy 83.82 252.73) (xy 83.82 248.92)
+			(xy 314.96 228.6) (xy 317.5 228.6)
 		)
 		(stroke
@@
 	(wire
 		(pts
-			(xy 314.96 228.6) (xy 317.5 228.6)
+			(xy 219.71 238.76) (xy 219.71 240.03)
 		)
 		(stroke
@@
 	(wire
 		(pts
-			(xy 217.17 238.76) (xy 218.44 238.76)
+			(xy 217.17 238.76) (xy 219.71 238.76)
 		)
 		(stroke
@@
 	(wire
 		(pts
-			(xy 176.53 245.11) (xy 170.18 245.11)
+			(xy 207.01 233.68) (xy 205.74 233.68)
 		)
 		(stroke
@@
 	(wire
 		(pts
-			(xy 218.44 238.76) (xy 218.44 234.95)
+			(xy 176.53 245.11) (xy 170.18 245.11)
 		)
 		(stroke
@@
 	(wire
 		(pts
-			(xy 205.74 228.6) (xy 205.74 238.76)
+			(xy 217.17 233.68) (xy 219.71 233.68)
 		)
 		(stroke
@@
 	(wire
 		(pts
+			(xy 205.74 238.76) (xy 205.74 243.84)
+		)
+		(stroke
+			(width 0)
+			(type default)
+		)
+	)
+	(wire
+		(pts
 			(xy 271.78 99.06) (xy 257.81 99.06)
 		)
@@
 	(wire
 		(pts
-			(xy 52.07 58.42) (xy 67.31 58.42)
+			(xy 207.01 238.76) (xy 205.74 238.76)
 		)
 		(stroke
@@
 	(wire
 		(pts
-			(xy 229.87 234.95) (xy 229.87 232.41)
+			(xy 52.07 58.42) (xy 67.31 58.42)
 		)
 		(stroke
@@
 	(wire
 		(pts
-			(xy 264.16 98.425) (xy 264.16 104.14)
+			(xy 229.87 234.95) (xy 229.87 232.41)
 		)
 		(stroke
@@
 	(wire
 		(pts
-			(xy 83.82 246.38) (xy 72.39 246.38)
+			(xy 264.16 98.425) (xy 264.16 104.14)
 		)
 		(stroke
@@
 	(wire
 		(pts
-			(xy 35.56 34.29) (xy 35.56 33.02)
+			(xy 83.82 246.38) (xy 72.39 246.38)
 		)
 		(stroke
@@
 	(wire
 		(pts
-			(xy 86.36 45.72) (xy 87.63 45.72)
+			(xy 35.56 34.29) (xy 35.56 33.02)
 		)
 		(stroke
@@
 	(wire
 		(pts
-			(xy 74.93 153.67) (xy 81.28 153.67)
+			(xy 86.36 45.72) (xy 87.63 45.72)
 		)
 		(stroke
@@
 	(wire
 		(pts
-			(xy 205.74 238.76) (xy 207.01 238.76)
+			(xy 74.93 153.67) (xy 81.28 153.67)
 		)
 		(stroke
@@
 	(wire
 		(pts
-			(xy 219.71 232.41) (xy 219.71 234.95)
+			(xy 219.71 232.41) (xy 219.71 233.68)
 		)
 		(stroke
@@
 	(wire
 		(pts
-			(xy 198.12 102.235) (xy 198.12 102.87)
+			(xy 205.74 233.68) (xy 205.74 228.6)
 		)
 		(stroke
@@
 	(wire
 		(pts
-			(xy 176.53 227.33) (xy 187.96 227.33)
-		)
-		(stroke
-			(width 0)
-			(type default)
-		)
-	)
-	(wire
-		(pts
-			(xy 204.47 233.68) (xy 207.01 233.68)
+			(xy 198.12 102.235) (xy 198.12 102.87)
 		)
 		(stroke
@@
 	(wire
 		(pts
-			(xy 218.44 234.95) (xy 219.71 234.95)
+			(xy 176.53 227.33) (xy 187.96 227.33)
 		)
 		(stroke
@@
 	(wire
 		(pts
+			(xy 219.71 233.68) (xy 219.71 234.95)
+		)
+		(stroke
+			(width 0)
+			(type default)
+		)
+	)
+	(wire
+		(pts
 			(xy 218.44 53.34) (xy 208.28 53.34)
 		)
@@
 	(wire
 		(pts
-			(xy 204.47 243.84) (xy 204.47 233.68)
-		)
-		(stroke
-			(width 0)
-			(type default)
-		)
-	)
-	(wire
-		(pts
 			(xy 86.36 45.72) (xy 85.09 45.72)
 		)
@@
 		)
 	)
+	(text "V05: \nC19, C20 Bump to 0805\nR2, R3 now 470 Ohm\nC22 Bump to 0603"
+		(exclude_from_sim no)
+		(at 376.936 69.088 0)
+		(effects
+			(font
+				(size 1.27 1.27)
+			)
+			(justify left)
+		)
+	)
 	(text "uC"
 		(exclude_from_sim no)
@@
 			)
 		)
-		(property "Value" "430"
+		(property "Value" "470"
 			(at 109.22 51.054 90)
 			(effects
@@
 			)
 		)
-		(property "Value" "430"
+		(property "Value" "470"
 			(at 109.22 60.96 90)
 			(effects
@@
 	(symbol
 		(lib_id "Device:Filter_EMI_LL_1423")
-		(at 212.09 236.22 180)
+		(at 212.09 236.22 0)
 		(unit 1)
 		(exclude_from_sim no)
@@
 		(dnp no)
 		(property "Reference" "FL1"
-			(at 212.471 243.84 0)
+			(at 211.709 228.6 0)
 			(effects
 				(font
@@
 		)
 		(property "Value" "ACT1210D-101-2P-TL00"
-			(at 209.55 241.554 0)
+			(at 214.63 230.886 0)
 			(effects
 				(font
@@
 		)
 		(property "Footprint" "_custom:ACT1210D1012PTL00"
-			(at 212.09 229.87 0)
+			(at 212.09 242.57 0)
 			(effects
 				(font
@@
 		)
 		(property "Datasheet" "~"
-			(at 212.09 237.236 90)
+			(at 212.09 235.204 90)
 			(effects
 				(font
@@
 			)
 		)
-		(property "Value" "2.2uF, X7R"
+		(property "Value" "2.2uF"
 			(at 283.718 168.402 0)
 			(effects
@@
 			)
 		)
-		(property "Footprint" "Capacitor_SMD:C_0402_1005Metric"
+		(property "Footprint" "Capacitor_SMD:C_0603_1608Metric"
 			(at 284.1752 170.18 0)
 			(effects
@@
 			)
 		)
-		(property "Footprint" "Capacitor_SMD:C_0603_1608Metric"
+		(property "Footprint" "Capacitor_SMD:C_0805_2012Metric"
 			(at 247.3452 170.18 0)
 			(effects
@@
 			)
 		)
-		(property "Footprint" "Capacitor_SMD:C_0603_1608Metric"
+		(property "Footprint" "Capacitor_SMD:C_0805_2012Metric"
 			(at 239.7252 170.18 0)
 			(effects

Commit message: big update
Parts:
- J5: value Conn_01x06_MountingPin -> Conn_Encoder
Connections:
- no-connect marks 36 -> 35
Other:
- moved on the sheet: C1, C10, C11, C12, C13, C2, C23, C24, C25, C3, C4, C5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
