File: 2. Little Boy - External (4.1A @ 36V)/1. Hardware/Little Boy - External.kicad_pcb (KiCad board)
At the start: 4 copper layers, 40 x 40 mm, 69 parts, among them J1 TESTPOINT, J10 MOT_B, J11 MOT_A, J12 TESTPOINT, J13 Control_In, J14 Control_In, J17 TESTPOINT, J2 TESTPOINT, J3 TESTPOINT, J5 Conn_01x06_MountingPin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

Commit message: v4 full
Parts:
- moved C10 0.75 mm to (161.2, 71.7)
Connections:
- J10 pad 2: (no net) -> Net-(J10-Pin_1)
Routing:
- net NRST: track 29.6 -> 29.1 mm
- net GND: track 22.6 -> 22.1 mm, vias 264 -> 267
